File: 2021-breadboard-power/2021-breadboard-power.sch (KiCad schematic (older format))
At the start: 11 parts, among them J1 PJ-102AH, J2 Conn_02x02_Odd_Even, J3 Conn_02x02_Odd_Even, U1 AZ1117CH-3.3TRG1, U2 AZ1117CH-5.0TRG1

Commit message: netlist
Parts:
- C1, C2, C3, C4: footprint (none) -> Capacitor_SMD:C_0805_2012Metric_Pad1.15x1.40mm_HandSolder
- D1: footprint (none) -> LED_THT:LED_D3.0mm
- J2, J3: footprint (none) -> Connector_PinHeader_2.54mm:PinHeader_2x02_P2.54mm_Vertical
- R1: footprint (none) -> Resistor_SMD:R_0805_2012Metric_Pad1.15x1.40mm_HandSolder
- U1, U2: footprint (none) -> Package_TO_SOT_SMD:SOT-223-3_TabPin2
Changed lines of the file:
@@
 F 0 "U1" H 4650 2983 50  0000 C CNN
 F 1 "AZ1117CH-3.3TRG1" H 4650 2892 50  0000 C CNN
-F 2 "" H 4650 2900 50  0001 C CIN
+F 2 "Package_TO_SOT_SMD:SOT-223-3_TabPin2" H 4650 2900 50  0001 C CIN
 F 3 "https://www.diodes.com/assets/Datasheets/AZ1117.pdf" H 4650 2650 50  0001 C CNN
 F 4 "AZ1117CH-3.3TRG1DICT-ND" H 4650 2801 50  0000 C CNN "digikey"
@@
 F 0 "U2" H 4650 4083 50  0000 C CNN
 F 1 "AZ1117CH-5.0TRG1" H 4650 3992 50  0000 C CNN
-F 2 "" H 4650 4000 50  0001 C CIN
+F 2 "Package_TO_SOT_SMD:SOT-223-3_TabPin2" H 4650 4000 50  0001 C CIN
 F 3 "https://www.diodes.com/assets/Datasheets/AZ1117.pdf" H 4650 3750 50  0001 C CNN
 F 4 "AZ1117CH-5.0TRG1DICT-ND" H 4650 3901 50  0000 C CNN "digikey"
@@
 F 0 "C1" H 3315 3041 50  0000 L CNN
 F 1 "10mF" H 3315 2950 50  0000 L CNN
-F 2 "" H 3238 2800 50  0001 C CNN
+F 2 "Capacitor_SMD:C_0805_2012Metric_Pad1.15x1.40mm_HandSolder" H 3238 2800 50  0001 C CNN
 F 3 "~" H 3200 2950 50  0001 C CNN
 F 4 "1276-6455-1-ND" H 3315 2859 50  0000 L CNN "digikey"
@@
 F 0 "C3" H 3315 4191 50  0000 L CNN
 F 1 "10mF" H 3315 4100 50  0000 L CNN
-F 2 "" H 3238 3950 50  0001 C CNN
+F 2 "Capacitor_SMD:C_0805_2012Metric_Pad1.15x1.40mm_HandSolder" H 3238 3950 50  0001 C CNN
 F 3 "~" H 3200 4100 50  0001 C CNN
 F 4 "1276-6455-1-ND" H 3315 4009 50  0000 L CNN "digikey"
@@
 F 0 "C2" H 6015 3041 50  0000 L CNN
 F 1 "22mF" H 6015 2950 50  0000 L CNN
-F 2 "" H 5938 2800 50  0001 C CNN
+F 2 "Capacitor_SMD:C_0805_2012Metric_Pad1.15x1.40mm_HandSolder" H 5938 2800 50  0001 C CNN
 F 3 "~" H 5900 2950 50  0001 C CNN
 F 4 "1276-6780-1-ND" H 6015 2859 50  0000 L CNN "digikey"
@@
 F 0 "C4" H 6015 4191 50  0000 L CNN
 F 1 "22mF" H 6015 4100 50  0000 L CNN
-F 2 "" H 5938 3950 50  0001 C CNN
+F 2 "Capacitor_SMD:C_0805_2012Metric_Pad1.15x1.40mm_HandSolder" H 5938 3950 50  0001 C CNN
 F 3 "~" H 5900 4100 50  0001 C CNN
 F 4 "1276-6780-1-ND" H 6015 4009 50  0000 L CNN "digikey"
@@
 F 0 "D1" H 4143 5366 50  0000 C CNN
 F 1 "LED" H 4143 5366 50  0001 C CNN
-F 2 "" H 4150 5150 50  0001 C CNN
+F 2 "LED_THT:LED_D3.0mm" H 4150 5150 50  0001 C CNN
 F 3 "~" H 4150 5150 50  0001 C CNN
 F 4 "732-5007-ND" H 4143 5275 50  0000 C CNN "digikey"
@@
 F 0 "R1" V 4850 5150 50  0000 C CNN
 F 1 "1k" V 4950 5150 50  0000 C CNN
-F 2 "" V 4880 5150 50  0001 C CNN
+F 2 "Resistor_SMD:R_0805_2012Metric_Pad1.15x1.40mm_HandSolder" V 4880 5150 50  0001 C CNN
 F 3 "~" H 4950 5150 50  0001 C CNN
 	1    4950 5150
@@
 F 0 "J3" H 7550 3700 50  0000 C CNN
 F 1 "Conn_02x02_Odd_Even" H 7550 4150 50  0001 C CNN
-F 2 "" H 7500 3900 50  0001 C CNN
+F 2 "Connector_PinHeader_2.54mm:PinHeader_2x02_P2.54mm_Vertical" H 7500 3900 50  0001 C CNN
 F 3 "~" H 7500 3900 50  0001 C CNN
 	1    7500 3900
@@
 F 0 "J2" H 7550 2600 50  0000 C CNN
 F 1 "Conn_02x02_Odd_Even" H 7550 3000 50  0001 C CNN
-F 2 "" H 7500 2800 50  0001 C CNN
+F 2 "Connector_PinHeader_2.54mm:PinHeader_2x02_P2.54mm_Vertical" H 7500 2800 50  0001 C CNN
 F 3 "~" H 7500 2800 50  0001 C CNN
 	1    7500 2800
