File: 1wamp-remake/1wamp-remake.kicad_pcb (KiCad board)
At the start: 2 copper layers, 10 parts, among them CN1 NMJ6HCD2, J1 Barrel_Jack_Switch

Commit message: updating
Parts:
- moved C1 126.7 mm to (26.2, 124.7), turned to 90 degrees
- moved C3 110.7 mm to (47.0, 118.1)
- moved R1 107.7 mm to (37.8, 124.2)
- moved D2 102.9 mm to (46.7, 141.5)
- moved CN1 99.2 mm to (32.3, 151.6), turned to 270 degrees
- moved J1 81.0 mm to (60.2, 137.4)
- moved R2 76.6 mm to (57.7, 125.0), turned to 270 degrees
- moved C2 75.3 mm to (45.7, 131.1)
- moved D1 73.8 mm to (56.1, 116.8)
- moved BT1 66.1 mm to (69.8, 139.7), turned to 180 degrees
Routing:
- net GND-B: track 0.00 -> 59.5 mm
- net GND-A: track 0.00 -> 36.7 mm
- net Net-(C3-Pad1): track 0.00 -> 28.5 mm
- net Net-(D1-Pad2): track 0.00 -> 28.0 mm
- net Net-(C1-Pad1): track 0.00 -> 25.3 mm
- net Net-(D2-Pad2): track 0.00 -> 14.9 mm
- net Net-(BT1-Pad1): track 0.00 -> 5.25 mm
- added copper zone on B.Cu, net GND-B
- added copper zone on F.Cu, net GND-B
Other:
- board outline added: 56.1 x 39.9 mm
